File: KiCad/MacroPad1.0/MacroPad1.1.kicad_pcb (KiCad board)
At the start: 2 copper layers, 76.7 x 45.2 mm, 28 parts, among them SW1 SW_Push, U1 ATmega32U4-A, Y1 16MHz

Commit message: Documentation Updates
Updated HTML BOM, small additions to README
Parts:
- C2, C3: value 1uF -> 14pF
Changed lines of the file:
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@@
       (effects (font (size 1 1) (thickness 0.15)) (justify mirror))
     )
-    (fp_text value "1uF" (at 0 -1.68 90) (layer "B.Fab")
+    (fp_text value "14pF" (at 0 -1.68 90) (layer "B.Fab")
       (effects (font (size 1 1) (thickness 0.15)) (justify mirror))
     )
@@
       (effects (font (size 1 1) (thickness 0.15)) (justify mirror))
     )
-    (fp_text value "1uF" (at 0 -1.68 90) (layer "B.Fab")
+    (fp_text value "14pF" (at 0 -1.68 90) (layer "B.Fab")
       (effects (font (size 1 1) (thickness 0.15)) (justify mirror))
     )
